File: BL-N305B/meshtastic-node.kicad_sch (KiCad schematic)
At the start: 116 parts, among them IC1 CH224K, IC2 CN3791, IC3 SKY65313-21, IC4 LR1110IMLTRT, J1 USB_C_Receptacle_USB2.0, J2 Conn_01x05_Socket, J3 Conn_Coaxial_Small, J4 Conn_01x02_Socket, J5 Conn_01x02_Socket, J6 Conn_ARM_JTAG_SWD_10, J7 Conn_Coaxial_Small, Q1 PMOS, Q2 PMOS, SW2 SW_Push, SW3 SW_DPDT_x2, U1 TPS565208, U2 TPS61222DCK, U3 TPS61220DCK, U4 BME280, U5 INA3221, U6 USBLC6-2SC6, U7 nRF52840, U8 BQ24650

Commit message: schematic
Parts:
- removed C1, C2, C3, C6, C7, C8: 10uF, Capacitor_SMD:C_0805_2012Metric_Pad1.18x1.45mm_HandSolder, symbol Device:C
- removed C4, C5: 100nF, Capacitor_SMD:C_0805_2012Metric_Pad1.18x1.45mm_HandSolder, symbol Device:C
- removed U7: nRF52840, Package_DFN_QFN:Nordic_AQFN-73-1EP_7x7mm_P0.5mm, symbol MCU_Nordic:nRF52840
- added C15, C49, C51: 4.7uF, Capacitor_SMD:C_0805_2012Metric_Pad1.18x1.45mm_HandSolder, symbol Device:C
- added C21, C31, C58, C59, C60, C61: 12pF, Capacitor_SMD:C_0805_2012Metric_Pad1.18x1.45mm_HandSolder, symbol Device:C
- added C32: 0.5pF, Capacitor_SMD:C_0805_2012Metric_Pad1.18x1.45mm_HandSolder, symbol Device:C
- added C33: 820pF, Capacitor_SMD:C_0805_2012Metric_Pad1.18x1.45mm_HandSolder, symbol Device:C
- added C46: 0.8pF, Capacitor_SMD:C_0805_2012Metric_Pad1.18x1.45mm_HandSolder, symbol Device:C
- added C47: 100pF, Capacitor_SMD:C_0805_2012Metric_Pad1.18x1.45mm_HandSolder, symbol Device:C
- added C48, C52, C53, C56: 100nF, Capacitor_SMD:C_0805_2012Metric_Pad1.18x1.45mm_HandSolder, symbol Device:C
- added C50, C54, C57: 1uF, Capacitor_SMD:C_0805_2012Metric_Pad1.18x1.45mm_HandSolder, symbol Device:C
- added C55: 47nF, Capacitor_SMD:C_0805_2012Metric_Pad1.18x1.45mm_HandSolder, symbol Device:C
- added L3: 15nH, Inductor_SMD:L_0805_2012Metric_Pad1.15x1.40mm_HandSolder, symbol Device:L
- added L4: 4.1nH, Inductor_SMD:L_0805_2012Metric_Pad1.15x1.40mm_HandSolder, symbol Device:L
- added L6, L7: 10uH, Inductor_SMD:L_0805_2012Metric_Pad1.15x1.40mm_HandSolder, symbol Device:L
- added U9: nRF52840, Package_DFN_QFN:Nordic_AQFN-73-1EP_7x7mm_P0.5mm, symbol MCU_Nordic:nRF52840
- added Y1, Y3: 32MHz, Crystal:Crystal_SMD_SeikoEpson_FA238V-4Pin_3.2x2.5mm, symbol Device:Crystal_GND2
- added Y2: 32.768kHz, Crystal:Crystal_SMD_SeikoEpson_FA238V-4Pin_3.2x2.5mm, symbol Device:Crystal_GND2
Connections:
- net D+: now also U9.AD6 (D+)
- net D-: now also U9.AD4 (D-)
- net GND: now also C15.2, C21.1, C31.1, C32.2, C33.2, C46.2, C47.2, C48.2, C49.2, C50.2, C51.2, C52.2, C53.2, C54.2, C55.2, C56.2, C57.2, C58.1, C59.1, C60.1, C61.1, U9.B7 (VSS), U9.EP (VSS), U9.F23 (VSS_PA), Y1.2, Y2.2, Y3.2
- net RF_WIFI_BT: now also C46.1, L4.2, U9.H23 (ANT); no longer AE1.1 (FEED)
- net RST: now also U9.AC13 (P0.18/~{RESET})
- net at IC4.7 (32K_P/_DIO11): now also C60.2
- net at IC4.8 (32K_N/_DIO10): now also C61.2, Y3.3
- new net: C21.2, U9.B24 (XC1), Y1.1
- new net: C58.2, U9.D2 (XL1/P0.00), Y2.3
- new net: C31.2, U9.A23 (XC2), Y1.3
- new net: C47.1, U9.D23 (DEC3)
- new net: L7.1, U9.AB2 (DCCH)
- new net: C48.1, U9.C1 (DEC1)
- new net: C15.1, U9.AC5 (DECUSB)
- new net: L6.2, U9.B3 (DCC)
- new net: C54.1, C55.1, L3.1, U9.B5 (DEC4), U9.E24 (DEC6)
- new net: C59.2, U9.F2 (XL2/P0.01), Y2.1
- new net: C33.1, U9.N24 (DEC5)
- new net: AE1.1 (FEED), C32.1, L4.1
- new net: L3.2, L6.1
- new net +1V8: C49.1, C51.1, C52.1, C53.1, C56.1, C57.1, L7.2, U9.A22 (VDD), U9.AD14 (VDD), U9.AD23 (VDD), U9.B1 (VDD), U9.W1 (VDD), U9.Y2 (VDDH)
- new net SWDC: U9.AA24 (SWDCLK)
- new net SWDI: U9.AC24 (SWDIO)
- new net VBUS_MAIN: C50.1, U9.AD2 (VBUS)
- no-connect marks 46 -> 16
Other:
- moved on the sheet: AE1, D2, R14, R16, R17, R24, SW2

Commit message: networks
Parts:
- removed C22, C23: 100nF, Capacitor_SMD:C_0805_2012Metric_Pad1.18x1.45mm_HandSolder, symbol Device:C
- removed R20: 100k, Resistor_SMD:R_0805_2012Metric_Pad1.20x1.40mm_HandSolder, symbol Device:R
- removed R21: 700k, Resistor_SMD:R_0805_2012Metric_Pad1.20x1.40mm_HandSolder, symbol Device:R
- removed U3: TPS61220DCK, Package_TO_SOT_SMD:Texas_R-PDSO-G6, symbol Regulator_Switching:TPS61222DCK
- removed U4: BME280, Package_LGA:Bosch_LGA-8_2.5x2.5mm_P0.65mm_ClockwisePinNumbering, symbol Sensor:BME280
- added C62: 100nF, Capacitor_SMD:C_0805_2012Metric_Pad1.18x1.45mm_HandSolder, symbol Device:C
- added C63: 470nF, Capacitor_SMD:C_0805_2012Metric_Pad1.18x1.45mm_HandSolder, symbol Device:C
- added C64, C65, C66, C67, C68, C69, C70, C71, C72, C73, C74, C75, C76, C77, C78, C80, C81, C82, C83: 12pF, Capacitor_SMD:C_0805_2012Metric_Pad1.18x1.45mm_HandSolder, symbol Device:C
- added J10, J9: Conn_Coaxial_Small, Connector_Coaxial:SMA_Molex_73251-1153_EdgeMount_Horizontal, symbol Connector:Conn_Coaxial_Small
- added L10, L11, L12, L13, L14, L15, L16, L17: 10uH, Inductor_SMD:L_0805_2012Metric_Pad1.15x1.40mm_HandSolder, symbol Device:L
- added L8: 15nH, Inductor_SMD:L_0805_2012Metric_Pad1.15x1.40mm_HandSolder, symbol Device:L
- added U3: AS179-92LF, Package_TO_SOT_SMD:SOT-363_SC-70-6, symbol RF_Switch:AS179-92LF
- added Y4: 32MHz, Crystal:Crystal_SMD_SeikoEpson_FA238V-4Pin_3.2x2.5mm, symbol Device:Crystal_GND2
- C34, C35: value 10uF -> 12pF
- C39: value 22uF -> 12pF
- L5: footprint Inductor_SMD:L_0805_2012Metric_Pad1.15x1.40mm_HandSolder -> Inductor_SMD:L_APV_ANR3010
- L9: value 4.7uH -> 10uH
- Y3: value 32MHz -> 32.768kHz
Connections:
- net +3V3: no longer C34.1, L9.1
- net +4V: no longer C35.1, C39.1
- net +5V: now also L16.2, L17.2
- net GND: now also C34.1, C35.1, C39.1, IC4.13 (GND_1), IC4.33 (GND_2), C62.2, C63.2, C64.1, C65.1, C68.2, C69.1, C70.1, C71.2, C72.1, C73.2, C76.2, C77.2, C80.2, C81.2, J10.2 (Ext), J9.2 (Ext), U3.2 (GND), Y4.2; no longer C34.2, C35.2, C39.2
- net VDD_RADIO: now also IC4.15 (VBAT), C62.1
- net at L9.2: now also C39.2, IC4.1 (VR_PA), C64.2, C65.2, L10.1
- net RF_SW3: now reaches IC4.10 (DIO8)
- net RF_SW2: now reaches IC4.11 (DIO7)
- net at IC4.12 (VREG): now also C63.1, L8.1
- net at IC4.14 (DCC_SW): now also L8.2
- net RF_SW1: now reaches IC4.19 (DIO6)
- net RF_SW1: now also U3.6 (V2)
- net RF_SW0: now reaches IC4.20 (DIO5)
- net RF_SW0: now also U3.4 (V1)
- net RADIO_SPI_MISO: now reaches IC4.21 (DIO4)
- net RADIO_SPI_MOSI: now reaches IC4.22 (DIO3)
- net RADIO_SPI_SCK: now reaches IC4.23 (DIO2)
- net RADIO_SPI_NSS: now reaches IC4.24 (DIO1)
- net RADIO_BUSY: now reaches IC4.25 (DIO0/BUSY)
- net at IC4.29 (RFI_N_LF0): now also C76.1, L13.1, L14.2
- net at IC4.30 (RFI_P_LF0): now also C78.2, L13.2
- net at IC4.31 (RFO_LP_LF): now also C66.2, L10.2, L12.1
- net at IC4.32 (RFO_HP_LF): now also L9.1, C67.1, L11.1
- net at IC4.4 (XTA): now also C34.2, Y4.1
- net at IC4.5 (XTB): now also C35.2, Y4.3
- net RADIO_RESET: now reaches IC4.6 (NRESET)
- net at C60.2, IC4.7 (32K_P/_DIO11): now also Y3.1
- net RADIO_IRQ: now reaches IC4.9 (DIO9)
- new net: C73.1, C75.1, U3.1 (J3)
- new net: C66.1, C68.1, C71.1, C75.2, L12.2
- new net: C81.1, C82.1, L15.1
- new net: C82.2, J9.1 (In), L16.1
- new net: C77.1, C78.1, C83.2, L14.1
- new net: C80.1, L15.2, U3.5 (J1)
- new net: C72.2, C74.2, U3.3 (J2)
- new net: C83.1, J10.1 (In), L17.1
- new net: C67.2, C69.2, C70.2, C74.1, L11.2
- no-connect marks 16 -> 19
Other:
- note added: "Bias Tee"
- note added: "Harmonic Filtering"
- note added: "Matching"
- note added: "PA Supply"
- note removed: "4V Boost"
- note removed: "ENVIRONMENT"
- note removed: "I2C ADDR 0x77"
- note removed: "SENSOR"
- moved on the sheet: C10, C11, C12, C13, C14, C16, C17, C18, C19, C20, C24, C37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
